File: pcb/reviung_ish_56_lp.kicad_sch (KiCad schematic)
At the start: 126 parts, among them J1 BAT, J2 BATTERY, SW1 POWER, SW2 RESET, U1 ProMicro

Commit message: WIP: switch to 2x1u space; experiment with straight bottom row
Parts:
- added D_G7: D, 42keebs:Diode_SOD123_dual_sided, symbol Device:D
- added SwG7: SW_Push, 42keebs:Kailh_socket_PG1350_1u_sw_cap, symbol Switch:SW_Push
- SwG2: footprint 42keebs:Kailh_socket_PG1350_1.5u_sw_cap -> 42keebs:Kailh_socket_PG1350_1u_sw_cap
Connections:
- net col2: now also SwG5.1
- net col3: now also SwG0.1; no longer SwG5.1
- net col4: now also SwG1.1; no longer SwG0.1
- net col5: now also SwG7.1; no longer SwG1.1
- net row4: now also D_G7.1 (K)
- new net: D_G7.2 (A), SwG7.2
Other:
- moved on the sheet: D_G0, D_G1, D_G5, SwG0, SwG1, SwG5
