File: pcb/rev57lp.kicad_sch (KiCad schematic)
At the start: 128 parts, among them J1 BAT, J2 BATTERY, SW1 POWER, SW2 RESET, U1 ProMicro

Commit message: Increase the angle of the sides to 15 degrees; update README
Parts:
- removed D_G7: D, 42keebs:Diode_SOD123_dual_sided, symbol Device:D
- removed SwG7: SW_Push, 42keebs:Kailh_socket_PG1350_1u_sw_cap, symbol Switch:SW_Push
- added D_GA2: D, 42keebs:Diode_SOD123_dual_sided, symbol Device:D
- added SwGA2: SW_Push, 42keebs:Kailh_socket_PG1350, symbol Switch:SW_Push
- H1, H2, H3, H4, H5, H6, H7, H8: footprint MountingHole:MountingHole_2.2mm_M2_ISO7380_Pad -> MountingHole:MountingHole_2.2mm_M2_Pad_Via; symbol Mechanical:MountingHole -> horizon-components:Hole_Pad
- J2: value BATTERY -> BAT; footprint Connector_JST:JST_PH_S2B-PH-K_1x02_P2.00mm_Horizontal -> Connector_PinHeader_2.54mm:PinHeader_1x02_P2.54mm_Vertical; now left out of the parts list
- SwA0, SwA1, SwA10, SwA11, SwA2, SwA3, SwA4, SwA5, SwA6, SwA7, SwA8, SwA9, SwB0, SwB1, SwB10, SwB11, SwB2, SwB3, SwB4, SwB5, SwB6, SwB7, SwB8, SwB9, SwC0, SwC1, SwC2, SwC3, SwC5, SwD0, SwD2, SwD3, SwD4, SwD5, SwD6, SwE0, SwE1, SwE2, SwE3, SwE4, SwE5, SwF0, SwF1, SwF2, SwF3, SwF4, SwF5, SwG0, SwG1, SwG3, SwG4, SwG5, SwG6: footprint 42keebs:Kailh_socket_PG1350_1u_sw_cap -> 42keebs:Kailh_socket_PG1350
- SwC4, SwD1: footprint 42keebs:Kailh_socket_PG1350_1u_sw_cap_home -> 42keebs:Kailh_socket_PG1350
- SwGB2: renamed from SwG2; footprint 42keebs:Kailh_socket_PG1350_1u_sw_cap -> 42keebs:Kailh_socket_PG1350
- renumbered D_G2 to D_GB2
Connections:
- net BAT: now also SW1.2 (B); no longer SW1.1 (A)
- net RAW: now also SW1.1 (A); no longer SW1.2 (B)
- net col5: now also SwGA2.1
- net row4: now also D_GA2.1 (K)
- new net: D_GA2.2 (A), SwGA2.2

Commit message: Bunch of modifications and tweaks:
* Drop the middle matrix column to free up one I/O pin
* Use dual DPDT switch symbol to fix DRC warnings about pins with no net
* Use standoff through holes instead of M2 mounting holes
Parts:
- added unit 2 of SW1
- H1, H2, H3, H4, H5, H6, H7, H8: footprint MountingHole:MountingHole_2.2mm_M2_Pad_Via -> 42keebs:MountingThroughHole_3.8mm_For_3mm_Standoff
- SW1: symbol Switch:SW_SPDT -> Switch:SW_DPDT_x2
- renumbered D_G5 to D_G0, D_G0 to D_G1, D_G1 to D_G2, D_GA2 to D_G3, D_D6 to D_G4, D_GB2 to D_G5, D_G3 to D_G6, D_G4 to D_G7, D_G6 to D_G8, SwG5 to SwG0, SwG0 to SwG1, SwG1 to SwG2, SwGA2 to SwG3, SwD6 to SwG4, SwGB2 to SwG5, SwG3 to SwG6, SwG4 to SwG7, SwG6 to SwG8
Connections:
- net col12 is gone; now on net col11: SwB11.1, SwB5.1, SwD5.1, SwF5.1, U1.12 (D9(PB5))
- net col10: now also SwB10.1, SwB4.1, SwD4.1, SwF4.1, SwG8.1, U1.11 (D8(PB4)); no longer SwB3.1, SwB9.1, SwD3.1, SwF3.1, U1.10 (D7(PE6))
- net col11: no longer SwB10.1, SwB4.1, SwD4.1, SwF4.1, U1.11 (D8(PB4))
- net col6: now also SwB0.1, SwB6.1, SwD0.1, SwF0.1, U1.7 (D4(PD4)); no longer SwG5.1, U1.6 (SCL(PD0))
- net col7: now also SwB1.1, SwB7.1, SwD1.1, SwF1.1, SwG5.1, U1.8 (D5(PC6)); no longer SwB0.1, SwB6.1, SwD0.1, SwF0.1, SwG6.1, U1.7 (D4(PD4))
- net col8: now also SwB2.1, SwB8.1, SwD2.1, SwF2.1, SwG6.1, U1.9 (D6(PD7)); no longer SwB1.1, SwB7.1, SwD1.1, SwF1.1, SwG7.1, U1.8 (D5(PC6))
- net col9: now also SwB3.1, SwB9.1, SwD3.1, SwF3.1, SwG7.1, U1.10 (D7(PE6)); no longer SwB2.1, SwB8.1, SwD2.1, SwF2.1, SwG8.1, U1.9 (D6(PD7))
- net row2: no longer D_G4.1 (K)
- net row4: now also D_G4.1 (K)
- new net RGB: U1.6 (SCL(PD0))
- no-connect marks 2 -> 5
Other:
- moved on the sheet: D_A0, D_A1, D_A10, D_A11, D_A2, D_A3, D_A4, D_A5, D_A6, D_A7, D_A8, D_A9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
